Commit message: urdf mesh 경로 상대경로로 지정

File: resources/robots/QUB/urdf/QUB.urdf (robot description, URDF)
Before this commit: robot QUB v1.2_urdf_4th, 14 links, 13 joints
Links:
- link L_ankle_link: geometry collision mesh filename=../meshes/L_ankle_link.STL; visual mesh filename=../meshes/L_ankle_link.STL
- link L_calf_link: geometry collision mesh filename=../meshes/L_calf_link.STL; visual mesh filename=../meshes/L_calf_link.STL
- link L_foot_link: geometry collision mesh filename=../meshes/L_foot_link.STL; visual mesh filename=../meshes/L_foot_link.STL
- link L_hip_r_link: geometry collision mesh filename=../meshes/L_hip_r_link.STL; visual mesh filename=../meshes/L_hip_r_link.STL
- link L_hip_y_link: geometry collision mesh filename=../meshes/L_hip_y_link.STL; visual mesh filename=../meshes/L_hip_y_link.STL
- link L_thigh_link: geometry collision mesh filename=../meshes/L_thigh_link.STL; visual mesh filename=../meshes/L_thigh_link.STL
- link R_ankle_link: geometry collision mesh filename=../meshes/R_ankle_link.STL; visual mesh filename=../meshes/R_ankle_link.STL
- link R_calf_link: geometry collision mesh filename=../meshes/R_calf_link.STL; visual mesh filename=../meshes/R_calf_link.STL
- link R_foot_link: geometry collision mesh filename=../meshes/R_foot_link.STL; visual mesh filename=../meshes/R_foot_link.STL
- link R_hip_r_link: geometry collision mesh filename=../meshes/R_hip_r_link.STL; visual mesh filename=../meshes/R_hip_r_link.STL
- link R_hip_y_link: geometry collision mesh filename=../meshes/R_hip_y_link.STL; visual mesh filename=../meshes/R_hip_y_link.STL
- link R_thigh_link: geometry collision mesh filename=../meshes/R_thigh_link.STL; visual mesh filename=../meshes/R_thigh_link.STL
- link base_link: geometry collision mesh filename=../meshes/base_link.STL; visual mesh filename=../meshes/base_link.STL
- link pelvis_link: geometry collision mesh filename=../meshes/pelvis_link.STL; visual mesh filename=../meshes/pelvis_link.STL

Commit message: 중력 문제, 발바닥 collision 문제 해결

File: resources/robots/QUB/urdf/QUB.urdf (robot description, URDF)
Before this commit: robot QUB v1.2_urdf_4th, 14 links, 13 joints
Links:
- link L_foot_link: geometry collision box size=0.12 0.06 0.04; visual mesh filename=../meshes/L_foot_link.STL
- link R_foot_link: geometry collision box size=0.12 0.06 0.04; visual mesh filename=../meshes/R_foot_link.STL

Commit message: collision 메쉬 파일 경로 재 지정

File: resources/robots/QUB/urdf/QUB.urdf (robot description, URDF)
Before this commit: robot QUB v1.2_urdf_4th, 14 links, 13 joints
Links:
- link L_ankle_link: geometry collision mesh filename=../meshes/collision/L_ankle_link.STL; visual mesh filename=../meshes/L_ankle_link.STL
- link L_calf_link: geometry collision mesh filename=../meshes/collision/L_calf_link.STL; visual mesh filename=../meshes/L_calf_link.STL
- link L_hip_r_link: geometry collision mesh filename=../meshes/collision/L_hip_r_link.STL; visual mesh filename=../meshes/L_hip_r_link.STL
- link L_hip_y_link: geometry collision mesh filename=../meshes/collision/L_hip_y_link.STL; visual mesh filename=../meshes/L_hip_y_link.STL
- link L_thigh_link: geometry collision mesh filename=../meshes/collision/L_thigh_link.STL; visual mesh filename=../meshes/L_thigh_link.STL
- link R_ankle_link: geometry collision mesh filename=../meshes/collision/R_ankle_link.STL; visual mesh filename=../meshes/R_ankle_link.STL
- link R_calf_link: geometry collision mesh filename=../meshes/collision/R_calf_link.STL; visual mesh filename=../meshes/R_calf_link.STL
- link R_hip_r_link: geometry collision mesh filename=../meshes/collision/R_hip_r_link.STL; visual mesh filename=../meshes/R_hip_r_link.STL
- link R_hip_y_link: geometry collision mesh filename=../meshes/collision/R_hip_y_link.STL; visual mesh filename=../meshes/R_hip_y_link.STL
- link R_thigh_link: geometry collision mesh filename=../meshes/collision/R_thigh_link.STL; visual mesh filename=../meshes/R_thigh_link.STL
- link base_link: geometry collision mesh filename=../meshes/collision/base_link.STL; visual mesh filename=../meshes/base_link.STL
- link pelvis_link: geometry collision mesh filename=../meshes/collision/pelvis_link.STL; visual mesh filename=../meshes/pelvis_link.STL

Commit message: RL 파일 수정

File: resources/robots/QUB/urdf/QUB.urdf (robot description, URDF)
Before this commit: robot QUB v1.2_urdf_4th, 14 links, 13 joints
Links:
- link L_ankle_link: mass 0.0236524344915325 -> 0.02200
- link L_calf_link: mass 1.17074765561419 -> 1.97157
- link L_foot_link: mass 0.359946537295079 -> 0.25200; geometry collision mesh filename=../meshes/collision/L_foot_link.STL; visual mesh filename=../meshes/L_foot_link.STL
- link L_hip_r_link: mass 0.855798957044734 -> 1.24854
- link L_hip_y_link: mass 0.917755275631564 -> 1.32879
- link L_thigh_link: mass 1.37472432263504 -> 2.18164
- link R_ankle_link: mass 0.0236524344915325 -> 0.02200
- link R_calf_link: mass 1.17074722849011 -> 1.97157
- link R_foot_link: mass 0.359946538045687 -> 0.25200; geometry collision mesh filename=../meshes/collision/R_foot_link.STL; visual mesh filename=../meshes/R_foot_link.STL
- link R_hip_r_link: mass 0.855799021923541 -> 1.24854
- link R_hip_y_link: mass 0.9177638118792 -> 1.32879
- link R_thigh_link: mass 1.3747257194995 -> 2.18164
- link base_link: mass 4.07254209371122 -> 4.21449; geometry collision box size=0.140 0.200 0.279; visual mesh filename=../meshes/base_link.STL
- link pelvis_link: mass 2.18597276276807 -> 3.69660

Commit message: 대칭구조 수정

File: resources/robots/QUB/urdf/QUB.urdf (robot description, URDF)
Before this commit: robot QUB, 14 links, 13 joints
Joints:
- joint R_ankle_pitch_joint: axis 0 -1 0 -> 0 1 0
- joint R_hip_pitch_joint: axis 0 1 0 -> 0 -1 0; limit lower=-1.5708 upper=0.5236 effort=60 velocity=5.0 -> lower=-0.5236 upper=1.5708 effort=60 velocity=5.0
- joint R_knee_pitch_joint: axis 0 -1 0 -> 0 1 0; limit lower=-1.9 upper=0.0 effort=120 velocity=5.0 -> lower=0.0 upper=1.9 effort=120 velocity=5.0
